File: stm32-battery.kicad_pcb (KiCad board)
At the start: 4 copper layers, 61 x 88.9 mm, 113 parts, among them J1 SWD, J2 Left, J3 Right, J4 Stemma I2C, J5 Micro SD, J6 USB-C, J7 DC In, J8 BATT, SW1 Reset, U1 STM32F103CBT6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

Commit message: jlcpcb order #, tooling, export
Parts:
- added REF**: JLCPCB-tooling-hole, local-footprints:JLCPCB-tooling-hole, F.Cu at (114.3, 134.6)
- added REF**: JLCPCB-tooling-hole, local-footprints:JLCPCB-tooling-hole, F.Cu at (114.3, 61.0)
- added REF**: JLCPCB-tooling-hole, local-footprints:JLCPCB-tooling-hole, F.Cu at (71.1, 134.6)
- added REF**: JLCPCB-tooling-hole, local-footprints:JLCPCB-tooling-hole, F.Cu at (71.1, 61.0)
Other:
- board text added: "JLCJLCJLCJLC"
Changed lines of the file:
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@@
   (title_block
     (title "STM32 with Battery")
-    (date "2022-09-14")
+    (date "2022-09-15")
     (rev "1")
     (company "#overviewer")
@@
     (pad_to_mask_clearance 0.05)
     (solder_mask_min_width 0.254)
+    (aux_axis_origin 62.23 142.24)
+    (grid_origin 62.23 142.24)
     (pcbplotparams
       (layerselection 0x00010fc_ffffffff)
       (disableapertmacros false)
-      (usegerberextensions false)
+      (usegerberextensions true)
       (usegerberattributes true)
       (usegerberadvancedattributes true)
@@
       (viasonmask false)
       (mode 1)
-      (useauxorigin false)
+      (useauxorigin true)
       (hpglpennumber 1)
       (hpglpenspeed 20)
@@
       (plotinvisibletext false)
       (sketchpadsonfab false)
-      (subtractmaskfromsilk false)
+      (subtractmaskfromsilk true)
       (outputformat 1)
       (mirror false)
-      (drillshape 1)
+      (drillshape 0)
       (scaleselection 1)
-      (outputdirectory "")
+      (outputdirectory "exported/")
     )
   )
@@
     (fp_line (start 1.6 0.8) (end -1.6 0.8) (layer "F.Fab") (width 0.1))
     (fp_line (start -1.6 -0.8) (end 1.6 -0.8) (layer "F.Fab") (width 0.1))
-    (pad "1" smd roundrect (at -1.475 0 180) (size 1.15 1.8) (layers "F.Cu" "F.Paste" "F.Mask") (roundrect_rratio 0.217391)
+    (pad "1" smd roundrect (at -1.475 0 180) (size 1.15 1.8) (layers "F.Cu" "F.Paste" "F.Mask") (roundrect_rratio 0.2173913043)
       (net 11 "+4V") (pintype "passive"))
-    (pad "2" smd roundrect (at 1.475 0 180) (size 1.15 1.8) (layers "F.Cu" "F.Paste" "F.Mask") (roundrect_rratio 0.217391)
+    (pad "2" smd roundrect (at 1.475 0 180) (size 1.15 1.8) (layers "F.Cu" "F.Paste" "F.Mask") (roundrect_rratio 0.2173913043)
       (net 2 "GND") (pintype "passive"))
     (model "${KICAD6_3DMODEL_DIR}/Capacitor_SMD.3dshapes/C_1206_3216Metric.wrl"
@@
     )
   )
+  (footprint "local-footprints:JLCPCB-tooling-hole" (layer "F.Cu")
+    (at 114.3 134.62)
+    (descr "Mounting Hole 2.1mm, no annular")
+    (tags "mounting hole 2.1mm no annular")
+    (attr exclude_from_pos_files exclude_from_bom)
+    (fp_text reference "REF**" (at 0 -3.2) (layer "F.SilkS") hide
+      (effects (font (size 1 1) (thickness 0.15)))
+    )
+    (fp_text value "JLCPCB-tooling-hole" (at 0 3.2) (layer "F.Fab")
+      (effects (font (size 1 1) (thickness 0.15)))
+    )
+    (fp_circle (center 0 0) (end 1.27 0) (layer "Cmts.User") (width 0.15) (fill none))
+    (fp_circle (center 0 0) (end 1.6 0) (layer "F.CrtYd") (width 0.05) (fill none))
+    (pad "" np_thru_hole circle (at 0 0) (size 1.152 1.152) (drill 1.152) (layers F&B.Cu *.Mask)
+      (solder_mask_margin 0.074) (clearance 1))
+  )
   (footprint "Jumper:SolderJumper-3_P1.3mm_Bridged12_RoundedPad1.0x1.5mm" (layer "F.Cu")
     (at 97.5 70.2575)
@@
       ))
   )
+  (footprint "local-footprints:JLCPCB-tooling-hole" (layer "F.Cu")
+    (at 114.3 60.96)
+    (descr "Mounting Hole 2.1mm, no annular")
+    (tags "mounting hole 2.1mm no annular")
+    (attr exclude_from_pos_files exclude_from_bom)
+    (fp_text reference "REF**" (at 0 -3.2) (layer "F.SilkS") hide
+      (effects (font (size 1 1) (thickness 0.15)))
+    )
+    (fp_text value "JLCPCB-tooling-hole" (at 0 3.2) (layer "F.Fab")
+      (effects (font (size 1 1) (thickness 0.15)))
+    )
+    (fp_circle (center 0 0) (end 1.27 0) (layer "Cmts.User") (width 0.15) (fill none))
+    (fp_circle (center 0 0) (end 1.6 0) (layer "F.CrtYd") (width 0.05) (fill none))
+    (pad "" np_thru_hole circle (at 0 0) (size 1.152 1.152) (drill 1.152) (layers F&B.Cu *.Mask)
+      (solder_mask_margin 0.074) (clearance 1))
+  )
   (footprint "Capacitor_SMD:C_0805_2012Metric" (layer "F.Cu")
     (at 103.925 114.9)
@@
     )
   )
+  (footprint "local-footprints:JLCPCB-tooling-hole" (layer "F.Cu")
+    (at 71.12 134.62)
+    (descr "Mounting Hole 2.1mm, no annular")
+    (tags "mounting hole 2.1mm no annular")
+    (attr exclude_from_pos_files exclude_from_bom)
+    (fp_text reference "REF**" (at 0 -3.2) (layer "F.SilkS") hide
+      (effects (font (size 1 1) (thickness 0.15)))
+    )
+    (fp_text value "JLCPCB-tooling-hole" (at 0 3.2) (layer "F.Fab")
+      (effects (font (size 1 1) (thickness 0.15)))
+    )
+    (fp_circle (center 0 0) (end 1.27 0) (layer "Cmts.User") (width 0.15) (fill none))
+    (fp_circle (center 0 0) (end 1.6 0) (layer "F.CrtYd") (width 0.05) (fill none))
+    (pad "" np_thru_hole circle (at 0 0) (size 1.152 1.152) (drill 1.152) (layers F&B.Cu *.Mask)
+      (solder_mask_margin 0.074) (clearance 1))
+  )
   (footprint "Jumper:SolderJumper-2_P1.3mm_Bridged_RoundedPad1.0x1.5mm" (layer "F.Cu")
     (at 89.2 89.624998 -90)
@@
     (fp_line (start 7.25 0.25) (end -1.25 0.25) (layer "F.Fab") (width 0.1))
     (fp_line (start 7.95 -1.35) (end 7.25 -1.35) (layer "F.Fab") (width 0.1))
-    (pad "1" thru_hole roundrect (at 0 0) (size 1.2 1.75) (drill 0.75) (layers *.Cu *.Mask) (roundrect_rratio 0.208333)
+    (pad "1" thru_hole roundrect (at 0 0) (size 1.2 1.75) (drill 0.75) (layers *.Cu *.Mask) (roundrect_rratio 0.2083333333)
       (net 27 "B10{slash}SCL") (pinfunction "SCL") (pintype "passive"))
     (pad "2" thru_hole oval (at 2 0) (size 1.2 1.75) (drill 0.75) (layers *.Cu *.Mask)
@@
     (fp_line (start 1.6 -0.8) (end 1.6 0.8) (layer "F.Fab") (width 0.1))
     (fp_line (start -1.6 -0.8) (end 1.6 -0.8) (layer "F.Fab") (width 0.1))
-    (pad "1" smd roundrect (at -1.475 0 180) (size 1.15 1.8) (layers "F.Cu" "F.Paste" "F.Mask") (roundrect_rratio 0.217391)
+    (pad "1" smd roundrect (at -1.475 0 180) (size 1.15 1.8) (layers "F.Cu" "F.Paste" "F.Mask") (roundrect_rratio 0.2173913043)
       (net 11 "+4V") (pintype "passive"))
-    (pad "2" smd roundrect (at 1.475 0 180) (size 1.15 1.8) (layers "F.Cu" "F.Paste" "F.Mask") (roundrect_rratio 0.217391)
+    (pad "2" smd roundrect (at 1.475 0 180) (size 1.15 1.8) (layers "F.Cu" "F.Paste" "F.Mask") (roundrect_rratio 0.2173913043)
       (net 2 "GND") (pintype "passive"))
     (model "${KICAD6_3DMODEL_DIR}/Capacitor_SMD.3dshapes/C_1206_3216Metric.wrl"
@@
     (fp_line (start -1.95 -1.35) (end -1.95 6.25) (layer "F.Fab") (width 0.1))
     (fp_line (start 3.25 0.25) (end -1.25 0.25) (layer "F.Fab") (width 0.1))
-    (pad "1" thru_hole roundrect (at 0 0 90) (size 1.2 1.75) (drill 0.75) (layers *.Cu *.Mask) (roundrect_rratio 0.208333)
+    (pad "1" thru_hole roundrect (at 0 0 90) (size 1.2 1.75) (drill 0.75) (layers *.Cu *.Mask) (roundrect_rratio 0.2083333333)
       (net 13 "+BATT") (pinfunction "Pin_1") (pintype "passive"))
     (pad "2" thru_hole oval (at 2 0 90) (size 1.2 1.75) (drill 0.75) (layers *.Cu *.Mask)
@@
     )
   )
+  (footprint "local-footprints:JLCPCB-tooling-hole" (layer "F.Cu")
+    (at 71.12 60.96)
+    (descr "Mounting Hole 2.1mm, no annular")
+    (tags "mounting hole 2.1mm no annular")
+    (attr exclude_from_pos_files exclude_from_bom)
+    (fp_text reference "REF**" (at 0 -3.2) (layer "F.SilkS") hide
+      (effects (font (size 1 1) (thickness 0.15)))
+    )
+    (fp_text value "JLCPCB-tooling-hole" (at 0 3.2) (layer "F.Fab")
+      (effects (font (size 1 1) (thickness 0.15)))
+    )
+    (fp_circle (center 0 0) (end 1.27 0) (layer "Cmts.User") (width 0.15) (fill none))
+    (fp_circle (center 0 0) (end 1.6 0) (layer "F.CrtYd") (width 0.05) (fill none))
+    (pad "" np_thru_hole circle (at 0 0) (size 1.152 1.152) (drill 1.152) (layers F&B.Cu *.Mask)
+      (solder_mask_margin 0.074) (clearance 1))
+  )
   (footprint "local-footprints:SWPA6020S" (layer "F.Cu")
     (at 110.125 110.3)
@@
     (effects (font (size 1 1) (thickness 0.15)))
   )
+  (gr_text "JLCJLCJLCJLC" (at 64.8 67.1 90) (layer "F.SilkS")
+    (effects (font (size 1 1) (thickness 0.15)))
+  )
