File: stm32-battery.kicad_sch (KiCad schematic)
At the start: 57 parts, among them J1 SWD, J2 Left, J3 Right, J4 Stemma I2C, J5 Micro SD, J6 USB-C, J7 DC In, J8 BATT, SW1 Reset, U1 STM32F103CBT6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

Commit message: part numbers for jst connectors / dc barrel jac
Parts:
- J4: Digikey # (none) -> S4B-PH-KL(LF)(SN)-ND
- J7: Mouser # (none) -> 992-CON-SOCJ-2155
- J8: Digikey # (none) -> S2B-PH-K-S(LF)(SN)
Changed lines of the file:
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@@
+      (effects (font (size 1.27 1.27)) hide)
+    )
+    (property "Digikey #" "S2B-PH-K-S(LF)(SN)" (id 4) (at 151.765 191.135 0)
       (effects (font (size 1.27 1.27)) hide)
     )
@@
       (effects (font (size 1.27 1.27)) hide)
     )
+    (property "Digikey #" "S4B-PH-KL(LF)(SN)-ND" (id 4) (at 248.92 137.16 0)
+      (effects (font (size 1.27 1.27)) hide)
+    )
     (pin "1")
     (pin "2")
@@
       (effects (font (size 1.27 1.27)) hide)
     )
+    (property "Mouser #" "992-CON-SOCJ-2155" (id 5) (at 127.635 182.245 0)
+      (effects (font (size 1.27 1.27)) hide)
+    )
